Commit message: Add Gazebo simulation support for E0509 with gripper
- Add gazebo.launch.py for standalone Gazebo simulation
- Add bringup_gazebo.launch.py for full simulation with RViz
- Add gz_controllers.yaml for ros2_control configuration
- Update URDF xacro with Gazebo-specific ros2_control
- Update CMakeLists.txt to install new files

File: urdf/e0509_with_gripper.urdf.xacro (robot description, xacro)
@@ -1,7 +1,7 @@
 <?xml version="1.0"?>
 <robot xmlns:xacro="http://www.ros.org/wiki/xacro" name="e0509_with_gripper">
-  <!-- Args (Doosan 스타일) -->
+  <!-- Arguments -->
   <xacro:arg name="color"        default="white"/>
-  <xacro:arg name="namespace"    default=""/>
+  <xacro:arg name="namespace"    default="e0509_gripper"/>
   <xacro:arg name="use_gazebo"   default="false"/>
   <xacro:arg name="host"         default="127.0.0.1"/>
@@ -12,5 +12,4 @@
   <xacro:arg name="update_rate"  default="100"/>
   <!-- Local properties -->
-  <xacro:property name="cr"          value="$(arg color)"/>
   <xacro:property name="gz"          value="$(arg use_gazebo)"/>
   <xacro:property name="host"        value="$(arg host)"/>
@@ -20,5 +19,5 @@
   <xacro:property name="model"       value="$(arg model)"/>
   <xacro:property name="update_rate" value="$(arg update_rate)"/>
-  <!-- Include E0509 macro (white) -->
+  <!-- Include E0509 macro (includes gazebo plugin) -->
   <xacro:include filename="$(find dsr_description2)/xacro/macro.e0509.white.xacro"/>
   <xacro:e0509 namespace="$(arg namespace)"/>
@@ -33,11 +32,47 @@
   <xacro:include filename="$(find rh_p12_rn_a_description)/urdf/rh_p12_rn_a.xacro"/>
   <xacro:rh_p12_rn_a prefix="gripper_"/>
-  <!-- Connect gripper to robot end-effector -->
-  <joint name="gripper_joint" type="fixed">
+  <!-- Connect gripper to robot -->
+  <joint name="gripper_attach_joint" type="fixed">
+    <origin xyz="0 0.0 0.0" rpy="0 0 0"/>
     <parent link="link_6"/>
     <child link="gripper_rh_p12_rn_base"/>
-    <origin xyz="0 0 0" rpy="0 0 0"/>
   </joint>
-  <!-- ros2_control (Doosan hardware interface) -->
+  <!-- Gazebo ros2_control -->
+  <xacro:if value="${gz}">
+    <!-- Arm ros2_control from dsr_description2 -->
+    <xacro:include filename="$(find dsr_description2)/ros2_control/e0509.gz_ros2_control.xacro"/>
+    <xacro:e0509_gz_ros2_control
+      name="e0509_gripper_gz"
+      namespace="$(arg namespace)"
+      update_rate="${update_rate}"
+    />
+    <!-- Gripper ros2_control - ALL 4 joints -->
+    <ros2_control name="gripper_gz" type="system">
+      <hardware>
+        <plugin>ign_ros2_control/IgnitionSystem</plugin>
+      </hardware>
+      <joint name="gripper_rh_r1">
+        <command_interface name="position"/>
+        <state_interface name="position"><param name="initial_value">0.0</param></state_interface>
+        <state_interface name="velocity"/>
+      </joint>
+      <joint name="gripper_rh_r2">
+        <command_interface name="position"/>
+        <state_interface name="position"><param name="initial_value">0.0</param></state_interface>
+        <state_interface name="velocity"/>
+      </joint>
+      <joint name="gripper_rh_l1">
+        <command_interface name="position"/>
+        <state_interface name="position"><param name="initial_value">0.0</param></state_interface>
+        <state_interface name="velocity"/>
+      </joint>
+      <joint name="gripper_rh_l2">
+        <command_interface name="position"/>
+        <state_interface name="position"><param name="initial_value">0.0</param></state_interface>
+        <state_interface name="velocity"/>
+      </joint>
+    </ros2_control>
+  </xacro:if>
+  <!-- Default ros2_control (Doosan hardware) -->
   <xacro:unless value="${gz}">
     <xacro:include filename="$(find dsr_description2)/ros2_control/e0509.ros2_control.xacro"/>
