Commit message: Add real gripper control via Tool Flange Serial (Modbus RTU)
- Add gripper.py: Real gripper control script using Modbus RTU protocol
- Update CMakeLists.txt: Install gripper.py
- Update README.md: Add real robot gripper control section with usage
- Fix gripper orientation in URDF (rotate 90 degrees)

🤖 Generated with [Claude Code](https://claude.com/claude-code)

Co-Authored-By: Claude Opus 4.5 <noreply@anthropic.com>

File: urdf/e0509_with_gripper.urdf.xacro (robot description, xacro)
@@ -34,5 +34,5 @@
   <!-- Connect gripper to robot -->
   <joint name="gripper_attach_joint" type="fixed">
-    <origin xyz="0 0.0 0.0" rpy="0 0 0"/>
+    <origin xyz="0 0.0 0.0" rpy="0 0 1.5708"/>
     <parent link="link_6"/>
     <child link="gripper_rh_p12_rn_base"/>
